File: lc_usb.kicad_pcb (KiCad board)
At the start: 2 copper layers, 67 x 24.7 mm, 32 parts, among them J1 USB_B_Mini, J2 Conn_01x02, J3 SPI, K1 FRT5, Q1 BC817, U1 AP1117-33, U2 ATMEGA8-16AU, U3 LM311, Y1 12Mhz

Commit message: minor changes
Connections:
- U3 pad 6: Net-(U3-Pad6) -> Net-(U3-Pad5)
Routing:
- net Net-(U3-Pad5): track 2.67 -> 8.80 mm
- net Net-(U3-Pad6): track 4.50 -> 0.00 mm
